Commit message: Extended URDF by another movable DOF.

File: urdf_kiba_example/urdf/myfirst.urdf (robot description, URDF)
Before this commit: robot myfirst, 4 links, 3 joints
Links:
- added link head_intermediate
Joints:
- removed joint head_to_base
- added joint head_to_base1: type continuous, parent base_link, child head_intermediate, origin xyz=0 0 0.3, axis 0 0 1
- added joint head_to_base2: type revolute, parent head_intermediate, child head, axis 1 0 0, limit lower=0.0 upper=0.7 effort=30 velocity=1.0
